File: mobo/Z.kicad_sch (KiCad schematic)
At the start: 12 parts, among them J110 Conn_01x04, U104 TMC2209-LA

Commit message: mobo v1, 1 unit
Parts:
- added R66, R67: 10k, symbol Device:R
- C25: renamed from C131; footprint (none) -> Capacitor_SMD:C_0603_1608Metric
- C26: renamed from C165; footprint (none) -> Capacitor_SMD:C_0402_1005Metric
- C29: renamed from C168; footprint (none) -> Capacitor_SMD:C_0402_1005Metric
- C30: renamed from C169; footprint (none) -> Capacitor_SMD:C_0402_1005Metric
- J7: renamed from J110; footprint (none) -> Connector_JST:JST_EH_B4B-EH-A_1x04_P2.50mm_Vertical
- renumbered C166 to C27, C167 to C28, C170 to C31, R128 to R10, R126 to R8, R127 to R9, U104 to U4
Connections:
- net GND: now also R66.1, R67.1
- net VDD: no longer U4.10 (MS2/AD1), U4.9 (MS1/AD0)
- net +24V: now reaches C26.2, C29.2, C30.2, C31.1, U4.22 (VS), U4.28 (VS)
- new net: R66.2, U4.9 (MS1/AD0)
- new net: R67.2, U4.10 (MS2/AD1)
- no-connect marks 2 -> 4
