File: mobo/mcu.kicad_sch (KiCad schematic)
At the start: 24 parts, among them SW101 SW_Push

Commit message: mobo v1, 1 unit
Parts:
- removed C108, C109, C110, C111, C112, C113, C114, C115, C116, C117, C118, C119, C120, C121: 100nF, symbol Device:C
- removed U115: ~, symbol mobo:_1
- added C10, C11, C13, C7, C8: 100nF, Capacitor_SMD:C_0402_1005Metric, symbol Device:C
- added FB2: FerriteBead, Inductor_SMD:L_0402_1005Metric, symbol Device:FerriteBead
- added R67: 10k, Resistor_SMD:R_0402_1005Metric, symbol Device:R
- added TP5: TestPoint, TestPoint:TestPoint_Pad_D2.0mm, symbol Connector:TestPoint
- added U2: STM32F405, mobo:LQFP-100_L14.0-W14.0-P0.50-LS16.0-BL, symbol mobo:STM32F405VGT
- C12: renamed from C103; footprint (none) -> Capacitor_SMD:C_0402_1005Metric
- C2: renamed from C102; value 0.1uF -> 100nF; footprint (none) -> Capacitor_SMD:C_0402_1005Metric
- C3: renamed from C104; footprint (none) -> Capacitor_SMD:C_0603_1608Metric
- C4: renamed from C105; footprint (none) -> Capacitor_SMD:C_0603_1608Metric
- C5: renamed from C106; footprint (none) -> Capacitor_SMD:C_0402_1005Metric
- C6: renamed from C107; footprint (none) -> Capacitor_SMD:C_0402_1005Metric
- C9: renamed from C101; footprint (none) -> Capacitor_SMD:C_0402_1005Metric
- R3: renamed from R101; footprint (none) -> Resistor_SMD:R_0402_1005Metric
- SW2: renamed from SW101; footprint (none) -> Button_Switch_SMD:SW_SPST_TS-1088-xR020
Connections:
- net GND: now also C10.2, C11.2, C13.2, C7.2, C8.2, U2.10 (VSS), U2.20 (VSSA), U2.27 (VSS), U2.74 (VSS), U2.99 (VSS)
- net NRST: now also R67.1, U2.14 (NRST)
- net VDDA: now also FB2.2, U2.21 (VREF+), U2.22 (VDDA)
- net at C4.2: now also U2.73 (VCAP_2)
- net at R3.1: now also TP5.1, U2.94 (BOOT0)
- net at C3.2: now also U2.49 (VCAP_1)
- net VDD renamed +3V3
- net +3V3: now also C10.1, C11.1, C13.1, C7.1, C8.1, FB2.1, R67.2, U2.100 (VDD), U2.11 (VDD), U2.19 (VDD), U2.28 (VDD), U2.50 (VDD), U2.6 (VBAT), U2.75 (VDD)
Other:
- moved on the sheet: C12, C2, C3, C4, C5, C6, C9, R3, SW2
