File: mobo/mcu_io.kicad_sch (KiCad schematic)
At the start: 5 parts, among them J102 SWD, Y101 8MHz

Commit message: mobo v1, 1 unit
Parts:
- removed J102: SWD, symbol Connector:Conn_01x06_Pin
- removed U115: ~, symbol mobo:_1
- added J20, J21: Conn_01x03, mobo:JST_PH_B3B-PH-SM4-TB_1x03-1MP_P2.00mm_Vertical, symbol Connector_Generic:Conn_01x03
- added J9: SWD, Connector_PinHeader_2.00mm:PinHeader_2x03_P2.00mm_Vertical, symbol Connector_Generic:Conn_02x03_Top_Bottom
- added U18: STM32G4A1CETx, Package_QFP:LQFP-48_7x7mm_P0.5mm, symbol MCU_ST_STM32G4:STM32G4A1CETx
- added U2: STM32F405, mobo:LQFP-100_L14.0-W14.0-P0.50-LS16.0-BL, symbol mobo:STM32F405VGT
- added U6: STM32H723VETx, Package_QFP:LQFP-100_14x14mm_P0.5mm, symbol MCU_ST_STM32H7:STM32H723VETx
- C67: renamed from C132; footprint (none) -> Capacitor_SMD:C_0402_1005Metric
- C68: renamed from C133; footprint (none) -> Capacitor_SMD:C_0402_1005Metric
- Y2: renamed from Y101; footprint (none) -> Crystal:Crystal_SMD_3225-4Pin_3.2x2.5mm
Connections:
- net D+: now also U2.70 (PA11)
- net D-: now also U2.69 (PA10)
- net GND: now also J20.2 (Pin_2), J21.2 (Pin_2), J9.5 (Pin_5)
- net NRST: now also J9.3 (Pin_3)
- net OSC_IN: now also U2.12 (PH0)
- net OSC_OUT: now also U2.13 (PH1)
- net PA0: now also U2.23 (PA0)
- net PA1: now also U2.24 (PA1)
- net PA2: now also U2.25 (PA2)
- net PA6: now also U2.31 (PA6)
- net PA7: now also U2.32 (PA7)
- net PB0: now also U2.35 (PB0)
- net PB1: now also U2.36 (PB1)
- net PB10: now also U2.47 (PB10)
- net PB13: now also U2.52 (PB13)
- net PB14: now also U2.53 (PB14)
- net PB15: now also U2.54 (PB15)
- net PB2: now also U2.37 (PB2)
- net PB3: now also U2.89 (PB3)
- net PB6: now also U2.92 (PB6)
- net PB7: now also U2.93 (PB7)
- net PB8: now also U2.95 (PB8)
- net PB9: now also U2.96 (PB9)
- net RX: now also U2.64 (PC7)
- net SWCLK: now also J9.2 (Pin_2), U2.76 (PA14)
- net SWDIO: now also J9.1 (Pin_1), U2.72 (PA13)
- net SWO: now also J9.6 (Pin_6)
- net TX: now also U2.63 (PC6)
- net VDD: now also J9.4 (Pin_4)
- net WIFI_EN: now also U2.62 (PD15)
- new net: U6.10 (VSS), U6.26 (VSS), U6.49 (VSS), U6.74 (VSS), U6.99 (VSS)
- new net: U18.23 (VSS), U18.35 (VSS), U18.47 (VSS)
- new net PA12: U2.71 (PA12)
- new net PA8: U2.67 (PA8)
- new net PA9: U2.68 (PA9)
- new net PB4: U2.90 (PB4)
- new net PB5: U2.91 (PB5)
- new net PC0: U2.15 (PC0)
- new net PC1: U2.16 (PC1)
- new net PC10: U2.78 (PC10)
- new net PC11: U2.79 (PC11)
- new net PC12: U2.80 (PC12)
- new net PC2: U2.17 (PC2)
- new net PC3: U2.18 (PC3)
- new net PC4: U2.33 (PC4)
- new net PC5: U2.34 (PC5)
- new net PC8: U2.65 (PC8)
- new net PC9: U2.66 (PC9)
- new net PD10: U2.57 (PD10)
- new net PD11: U2.58 (PD11)
- new net PD6: U2.87 (PD6)
- new net PD7: U2.88 (PD7)
- new net PD8: U2.55 (PD8)
- new net PD9: U2.56 (PD9)
- new net PE10: U2.41 (PE10)
- new net PE11: U2.42 (PE11)
- new net PE12: U2.43 (PE12)
- new net PE13: U2.44 (PE13)
- new net PE14: U2.45 (PE14)
- new net PE15: U2.46 (PE15)
- new net PE7: U2.38 (PE7)
- new net PE8: U2.39 (PE8)
- new net PE9: U2.40 (PE9)
- new net VCC: J20.3 (Pin_3), J21.3 (Pin_3)
- new net X_LIMIT: J20.1 (Pin_1), U2.81 (PD0)
- new net Y_LIMIT: J21.1 (Pin_1), U2.82 (PD1)
- no-connect marks 0 -> 17
Other:
- note removed: "tim2: x step, y step, lights tim3: z tim4: c tim5: c contd."
- moved on the sheet: C67, C68, Y2
