File: mobo/mobo.kicad_sch (KiCad schematic)
At the start: 11 parts, among them J104 X Axis, J105 Y Axis, J107 Encoders

Commit message: mobo v1, 1 unit
Parts:
- removed J104: X Axis, symbol Connector_Generic:Conn_01x03
- removed J105: Y Axis, symbol Connector_Generic:Conn_01x03
- removed J107: Encoders, symbol Connector_Generic:Conn_01x04
- added J24: Conn_01x06, Connector_JST:JST_XH_B6B-XH-A_1x06_P2.50mm_Vertical, symbol Connector_Generic:Conn_01x06
- added J3: Conn_01x07, Connector_JST:JST_XH_B7B-XH-A_1x07_P2.50mm_Vertical, symbol Connector_Generic:Conn_01x07
- added J5: SPI, Connector_JST:JST_EH_S3B-EH_1x03_P2.50mm_Horizontal, symbol Connector_Generic:Conn_01x03
- H2: renamed from H101; footprint (none) -> MountingHole:MountingHole_2.2mm_M2_Pad_Via
- H3: renamed from H102; footprint (none) -> MountingHole:MountingHole_2.2mm_M2_Pad_Via
- H4: renamed from H103; footprint (none) -> MountingHole:MountingHole_2.2mm_M2_Pad_Via
- H5: renamed from H104; footprint (none) -> MountingHole:MountingHole_2.2mm_M2_Pad_Via
- R2: renamed from R151; footprint (none) -> Resistor_SMD:R_0402_1005Metric
- renumbered FID101 to FID2, FID102 to FID3, FID103 to FID4
Connections:
- net GND: now also J24.6 (Pin_6)
- net MCU - IO/PB10 renamed MCU - IO/PC10
- net PDN_UART renamed UART_C
- new net MCU - IO/PA12: J24.5 (Pin_5)
- new net MCU - IO/PA8: J24.3 (Pin_3)
- new net MCU - IO/PA9: J24.1 (Pin_1)
- new net MCU - IO/PB13: J3.1 (Pin_1)
- new net MCU - IO/PB14: J3.2 (Pin_2)
- new net MCU - IO/PB15: J3.3 (Pin_3)
- new net MCU - IO/PB3: J5.3 (Pin_3)
- new net MCU - IO/PB4: J5.2 (Pin_2)
- new net MCU - IO/PB5: J5.1 (Pin_1)
- new net MCU - IO/PC8: J24.4 (Pin_4)
- new net MCU - IO/PC9: J24.2 (Pin_2)
- new net MCU - IO/PD10: J3.6 (Pin_6)
- new net MCU - IO/PD11: J3.7 (Pin_7)
- new net MCU - IO/PD8: J3.4 (Pin_4)
- new net MCU - IO/PD9: J3.5 (Pin_5)
Other:
- removed sheet Feeders
- sheet C1: file C.kicad_sch -> motor_driver.kicad_sch
- sheet C2: file C.kicad_sch -> motor_driver.kicad_sch
- sheet C3: file C.kicad_sch -> motor_driver.kicad_sch
- sheet C4: file C.kicad_sch -> motor_driver.kicad_sch
- sheet C5: file C.kicad_sch -> motor_driver.kicad_sch
- sheet C6: file C.kicad_sch -> motor_driver.kicad_sch
- sheet MCU - IO ports: added PA12, PA8, PA9, PB13, PB14, PB15, PB3, PB4, PB5, PC10, PC11, PC12, PC4, PC5, PC8, PC9, PD10, PD11, PD8, PD9, PE10, PE11, PE12, PE13, PE14, PE9; removed PA3, PA4, PA5, PA6, PA7, PB0, PB1, PB11, PB12
- sheet Power ports: added none; removed LDO_EN
- sheet Z1: file Z.kicad_sch -> motor_driver.kicad_sch
- sheet Z2: file Z.kicad_sch -> motor_driver.kicad_sch
- sheet Z3: file Z.kicad_sch -> motor_driver.kicad_sch
- note added: "CHECK EVERYTHING"
- note added: "PCB editor"
- note added: "To external toolhead"
- note added: "driver sections route on mobo"
- note added: "finish the entire driver board, like route it too"
- note added: "footprints"
- note added: "light pcb"
- note added: "limit switches finish r/c stuff test points status leds"
- note added: "make / outline a plan for how it communicates"
- note removed: "finish all the pin assignments"
- note removed: "finish the x and y board"
- note removed: "make a table with all the pin assignments"
- moved on the sheet: FID2, FID3, FID4, H2, H3, H4, H5, R2
