File: mobo/motor_driver.kicad_sch (KiCad schematic)
At the start: 14 parts, among them J10 Conn_01x04, U7 TMC2209-LA

Commit message: mobo v1, 1 unit
Parts:
- C25: renamed from C46; footprint (none) -> Capacitor_SMD:C_0603_1608Metric
- C26: renamed from C47; footprint (none) -> Capacitor_SMD:C_0402_1005Metric
- C27: renamed from C48; footprint (none) -> Capacitor_SMD:C_0805_2012Metric
- C28: renamed from C50; footprint (none) -> Capacitor_SMD:C_0603_1608Metric
- C29: renamed from C49; footprint (none) -> Capacitor_SMD:C_0402_1005Metric
- C30: renamed from C51; footprint (none) -> Capacitor_SMD:C_0402_1005Metric
- C31: renamed from C52; footprint (none) -> Capacitor_SMD:CP_Elec_6.3x5.8
- J7: renamed from J10; footprint Connector_JST:JST_EH_B4B-EH-A_1x04_P2.50mm_Vertical -> mobo:JST_PH_B4B-PH-SM4-TB_1x04-1MP_P2.00mm_Vertical
- R10: renamed from R19; footprint (none) -> Resistor_SMD:R_0402_1005Metric
- R14: renamed from R20; footprint (none) -> Resistor_SMD:R_1206_3216Metric
- R15: renamed from R21; footprint (none) -> Resistor_SMD:R_1206_3216Metric
- R8: renamed from R17; footprint (none) -> Resistor_SMD:R_0402_1005Metric
- R9: renamed from R18; footprint (none) -> Resistor_SMD:R_0402_1005Metric
- U4: renamed from U7; footprint Package_DFN_QFN:VQFN-28-1EP_5x5mm_P0.5mm_EP3.7x3.7mm_ThermalVias -> mobo:VQFN-28-1EP_5x5mm_P0.5mm_EP3.7x3.7mm_ThermalVias
Connections:
- net VCC renamed +3V3
