File: mobo/power.kicad_sch (KiCad schematic)
At the start: 64 parts, among them J103 PSU, Q103 NMOS, Q104 NMOS, U105 TPS54302, U106 LM5146RGYR, U107 TLV75533PDBV

Commit message: mobo v1, 1 unit
Parts:
- removed C141, C142: 1uF, symbol Device:C
- removed J103: PSU, symbol Connector_Generic:Conn_01x02
- removed Q103: NMOS, symbol Simulation_SPICE:NMOS
- removed TP103: TestPoint, symbol Connector:TestPoint
- removed U107: TLV75533PDBV, Package_TO_SOT_SMD:SOT-23-5, symbol Regulator_Linear:TLV75533PDBV
- added C119: 10uF, Capacitor_SMD:C_0805_2012Metric, symbol Device:C
- added C120: 22uF, Capacitor_SMD:C_0805_2012Metric, symbol Device:C
- added D6: 15V, Diode_SMD:D_SOD-123F, symbol Device:D_Zener
- added D7: D_TVS, Diode_SMD:D_SMC, symbol Device:D_TVS
- added F1: Fuse, Fuse:Fuseholder_Littelfuse_Nano2_154x, symbol Device:Fuse
- added J13: PSU, TerminalBlock_Phoenix:TerminalBlock_Phoenix_MKDS-1,5-2-5.08_1x02_P5.08mm_Horizontal, symbol Connector:Screw_Terminal_01x02
- added L4: 2.2uH, Inductor_SMD:L_APV_ANR3012, symbol Device:L
- added Q2: C478471, Package_SON:VSON-8_3.3x3.3mm_P0.65mm_NexFET, symbol Simulation_SPICE:NMOS
- added Q4: PMOS, Package_TO_SOT_SMD:TO-252-2_TabPin1, symbol Simulation_SPICE:PMOS
- added R63: 100k, Resistor_SMD:R_0603_1608Metric, symbol Device:R
- added R68, R69: 0, Resistor_SMD:R_0603_1608Metric, symbol Device:R
- added R70: 100k, Resistor_SMD:R_0402_1005Metric, symbol Device:R
- added TP4, TP6, TP7, TP8: TestPoint, TestPoint:TestPoint_Pad_D2.0mm, symbol Connector:TestPoint
- added U17: TPS62160DGK, Package_SO:MSOP-8_3x3mm_P0.65mm, symbol Regulator_Switching:TPS62160DGK
- C100: renamed from C152; footprint (none) -> Capacitor_SMD:C_1210_3225Metric
- C101: renamed from C157; footprint (none) -> Capacitor_SMD:C_1210_3225Metric
- C102: renamed from C144; value 100pF -> 150pF; footprint (none) -> Capacitor_SMD:C_0402_1005Metric
- C103: renamed from C158; footprint (none) -> Capacitor_SMD:C_1210_3225Metric
- C104: renamed from C143; footprint (none) -> Capacitor_SMD:C_0402_1005Metric
- C105: renamed from C159; footprint (none) -> Capacitor_SMD:C_1210_3225Metric
- C106: renamed from C140; footprint (none) -> Capacitor_SMD:C_0603_1608Metric
- C107: renamed from C160; footprint (none) -> Capacitor_SMD:C_1210_3225Metric
- C108: renamed from C136; footprint (none) -> Capacitor_SMD:C_0603_1608Metric
- C109: renamed from C161; footprint (none) -> Capacitor_SMD:C_1210_3225Metric
- C110: renamed from C162; footprint (none) -> Capacitor_SMD:C_1210_3225Metric
- C111: renamed from C137; footprint (none) -> Capacitor_SMD:C_1210_3225Metric
- C112: renamed from C147; footprint (none) -> Capacitor_SMD:C_0603_1608Metric
- C113: renamed from C163; footprint (none) -> Capacitor_SMD:C_1210_3225Metric
- C114: renamed from C138; footprint (none) -> Capacitor_SMD:C_1210_3225Metric
- C115: renamed from C139; footprint (none) -> Capacitor_SMD:C_0603_1608Metric
- C116: renamed from C164; footprint (none) -> Capacitor_SMD:C_1210_3225Metric
- C117: renamed from C146; footprint (none) -> Capacitor_SMD:C_0603_1608Metric
- C118: renamed from C145; footprint (none) -> Capacitor_SMD:C_0805_2012Metric
- C90: renamed from C149; footprint (none) -> Capacitor_SMD:C_1210_3225Metric
- C91: renamed from C153; footprint (none) -> Capacitor_SMD:C_1210_3225Metric
- C92: renamed from C154; footprint (none) -> Capacitor_SMD:C_1210_3225Metric
- C93: renamed from C150; footprint (none) -> Capacitor_SMD:C_1210_3225Metric
- C94: renamed from C134; footprint (none) -> Capacitor_SMD:C_1210_3225Metric
- C95: renamed from C155; footprint (none) -> Capacitor_SMD:C_1210_3225Metric
- C96: renamed from C151; footprint (none) -> Capacitor_SMD:C_1210_3225Metric
- C97: renamed from C135; footprint (none) -> Capacitor_SMD:C_0603_1608Metric
- C98: renamed from C156; footprint (none) -> Capacitor_SMD:C_1210_3225Metric
- C99: renamed from C148; footprint (none) -> Capacitor_SMD:C_0402_1005Metric
- D2: renamed from D101; footprint (none) -> LED_SMD:LED_0805_2012Metric
- D3: renamed from D104; footprint (none) -> LED_SMD:LED_0805_2012Metric
- D4: renamed from D102; footprint (none) -> LED_SMD:LED_0805_2012Metric
- D5: renamed from D103; footprint (none) -> LED_SMD:LED_0805_2012Metric
- L2: renamed from L101; footprint (none) -> Inductor_SMD:L_SOREDE_SNR.1050_10x10x5mm
- L3: renamed from L102; footprint (none) -> Inductor_SMD:L_Ferrocore_DLG-1004
- Q3: renamed from Q104; value NMOS -> C3011225; footprint (none) -> Package_DFN_QFN:PQFN-8-EP_6x5mm_P1.27mm_Generic
- R47: renamed from R120; footprint (none) -> Resistor_SMD:R_0402_1005Metric
- R48: renamed from R107; value 511k -> 510k; footprint (none) -> Resistor_SMD:R_0603_1608Metric
- R49: renamed from R108; footprint (none) -> Resistor_SMD:R_0603_1608Metric
- R50: renamed from R121; footprint (none) -> Resistor_SMD:R_0402_1005Metric
- R51: renamed from R119; footprint (none) -> Resistor_SMD:R_0402_1005Metric
- R52: renamed from R118; footprint (none) -> Resistor_SMD:R_0402_1005Metric
- R53: renamed from R112; footprint (none) -> Resistor_SMD:R_0402_1005Metric
- R54: renamed from R117; footprint (none) -> Resistor_SMD:R_0402_1005Metric
- R55: renamed from R113; footprint (none) -> Resistor_SMD:R_0603_1608Metric
- R56: renamed from R122; footprint (none) -> Resistor_SMD:R_0402_1005Metric
- R57: renamed from R109; footprint (none) -> Resistor_SMD:R_0603_1608Metric
- R58: renamed from R110; footprint (none) -> Resistor_SMD:R_0603_1608Metric
- R59: renamed from R111; footprint (none) -> Resistor_SMD:R_0603_1608Metric
- R60: renamed from R123; footprint (none) -> Resistor_SMD:R_0805_2012Metric
- R61: renamed from R114; footprint (none) -> Resistor_SMD:R_1206_3216Metric
- R62: renamed from R124; value 10k -> 4.7k; footprint (none) -> Resistor_SMD:R_0805_2012Metric
- R64: renamed from R115; value 4.7k -> 560R; footprint (none) -> Resistor_SMD:R_0603_1608Metric
- R65: renamed from R116; value 1k -> 220R; footprint (none) -> Resistor_SMD:R_0603_1608Metric
- TP2: renamed from TP101; footprint (none) -> TestPoint:TestPoint_Pad_D2.0mm
- TP3: renamed from TP102; footprint (none) -> TestPoint:TestPoint_Pad_D2.0mm
- renumbered U105 to U15, U106 to U16
Connections:
- net +24V: now also TP6.1
- net GND: now also C119.2, C120.2, J13.1 (Pin_1), R70.2, TP7.1, U17.1 (PGND), U17.4 (AGND)
- net at U16.18 (HO): now also Q2.2 (G)
- net at C108.2, L2.1, U15.2 (SW): now also TP8.1
- net at U15.6 (BOOT): now also R68.1; no longer C108.1
- net at R57.2, R58.1: now also R69.2; no longer C115.2
- net Cin: no longer names the net of C117.1, L3.1, Q3.1 (D), R60.1, U16.19 (SW)
- net Cin: now also Q2.3 (S); no longer C100.1, C90.1, C93.1, C96.1
- net VCC renamed +3V3
- net +3V3: now also C120.1, L4.2, R63.1, TP4.1, U17.6 (VOS)
- net VDC renamed +48V
- net +48V: now also C100.1, C90.1, C93.1, C96.1, Q2.1 (D), Q4.1 (D)
- net VDD renamed +5V
- net +5V: now also C119.1, U17.2 (VIN), U17.3 (EN)
- new net: C108.1, R68.2
- new net: D7.1 (A1), F1.2
- new net: D6.2 (A), Q4.2 (G), R70.1
- new net: D6.1 (K), D7.2 (A2), Q4.3 (S)
- new net: L4.1, U17.7 (SW)
- new net: C115.2, R69.1
- new net GNDA: U17.5 (FB)
- new net PG: R63.2, U17.8 (PG)
- new net POWER_SUPPLY: F1.1, J13.2 (Pin_2)
Other:
- note added: "CVIN"
- note added: "RVIN"
- note added: "check l2"
- note removed: "24V"
- note removed: "3.3V"
- note removed: "48V"
- note removed: "5V"
- note removed: "Status LEDs"
- moved on the sheet: C100, C101, C102, C103, C104, C105, C106, C107, C108, C109, C110, C111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
