File: mobo/wifi.kicad_sch (KiCad schematic)
At the start: 5 parts, among them U102 ESP32-WROOM-32E

Commit message: mobo v1, 1 unit
Parts:
- C23: renamed from C122; footprint (none) -> Capacitor_SMD:C_0805_2012Metric
- C24: renamed from C123; footprint (none) -> Capacitor_SMD:C_0402_1005Metric
- R4: renamed from R102; footprint (none) -> Resistor_SMD:R_0402_1005Metric
- R5: renamed from R103; footprint (none) -> Resistor_SMD:R_0402_1005Metric
- renumbered U102 to U3
Connections:
- net VCC renamed +3V3
